File: Schematics/JJ65c02/JJ65c02_support.kicad_sch (KiCad schematic)
At the start: 28 parts, among them SW2 SW_SPDT, U1 74HC00, U3 TXB0108PWR, U4 TXB0104PW, U5 74LS573, U6 TLV2217-33KCSE3, X1 1.8Mhz

Commit message: Some updates for true 2.0.0 release
Parts:
- DECODER1: value 22V10C -> ATF22V10C-7
Changed lines of the file:
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@@
 		(on_board yes)
 		(dnp no)
-		(fields_autoplaced yes)
 		(property "Reference" "DECODER1"
-			(at 186.69 69.6427 0)
+			(at 185.928 69.342 0)
 			(effects
 				(font
@@
 			)
 		)
-		(property "Value" "22V10C"
-			(at 186.69 72.0669 0)
+		(property "Value" "ATF22V10C-7"
+			(at 186.436 71.628 0)
 			(effects
 				(font

Commit message: Schematic changes - Banking
Connections:
- net SND: now also AUDIO1.R, AUDIO1.T, C11.2, C12.1, C12.2, R4.1, R5.2, R6.2
- net BK2: now reaches DECODER1.11 (IN11)
- net BA16: now reaches DECODER1.18 (IO17)
- no-connect marks 38 -> 36
Other:
- moved on the sheet: POWER1
Changed lines of the file:
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@@
 	)
 	(no_connect
-		(at 173.99 101.6)
-	)
-	(no_connect
-		(at 199.39 91.44)
-	)
-	(no_connect
 		(at 39.37 35.56)
 	)
@@
 	(wire
 		(pts
-			(xy 153.67 46.99) (xy 162.56 46.99)
+			(xy 153.67 49.53) (xy 162.56 49.53)
 		)
 		(stroke
@@
 		)
 		(stroke
-			(width 0)
+			(width 0.2032)
 			(type default)
 		)
@@
 		)
 		(stroke
-			(width 0)
+			(width 0.2032)
 			(type default)
 		)
@@
 		)
 		(stroke
-			(width 0)
+			(width 0.2032)
 			(type default)
 		)
@@
 		)
 		(stroke
-			(width 0)
+			(width 0.2032)
 			(type default)
 		)
@@
 		)
 		(stroke
-			(width 0)
+			(width 0.2032)
 			(type default)
 		)
@@
 		)
 		(stroke
-			(width 0)
+			(width 0.2032)
 			(type default)
 		)
@@
 	(wire
 		(pts
-			(xy 162.56 46.99) (xy 162.56 44.45)
+			(xy 162.56 49.53) (xy 162.56 46.99)
 		)
 		(stroke
@@
 		)
 		(stroke
-			(width 0)
+			(width 0.2032)
 			(type default)
 		)
@@
 		)
 		(stroke
-			(width 0)
+			(width 0.2032)
 			(type default)
 		)
@@
 	(wire
 		(pts
+			(xy 171.45 101.6) (xy 173.99 101.6)
+		)
+		(stroke
+			(width 0)
+			(type default)
+		)
+	)
+	(wire
+		(pts
 			(xy 76.2 180.34) (xy 78.74 180.34)
 		)
@@
 		)
 		(stroke
-			(width 0)
+			(width 0.2032)
 			(type default)
 		)
@@
 		)
 		(stroke
-			(width 0)
+			(width 0.2032)
 			(type default)
 		)
@@
 	(wire
 		(pts
+			(xy 162.56 36.83) (xy 162.56 39.37)
+		)
+		(stroke
+			(width 0.3048)
+			(type default)
+		)
+	)
+	(wire
+		(pts
 			(xy 44.45 157.48) (xy 50.8 157.48)
 		)
@@
 		)
 		(stroke
-			(width 0)
+			(width 0.2032)
 			(type default)
 		)
@@
 		)
 	)
+	(wire
+		(pts
+			(xy 199.39 91.44) (xy 201.93 91.44)
+		)
+		(stroke
+			(width 0)
+			(type default)
+		)
+	)
 	(bus
 		(pts
@@
 		)
 	)
+	(label "SND"
+		(at 128.27 153.67 0)
+		(effects
+			(font
+				(size 1.1938 1.1938)
+			)
+			(justify left bottom)
+		)
+	)
 	(label "d3v0"
 		(at 238.76 120.65 180)
@@
 		)
 	)
+	(label "SND"
+		(at 152.4 153.67 0)
+		(effects
+			(font
+				(size 1.1938 1.1938)
+			)
+			(justify left bottom)
+		)
+	)
 	(label "d3v7"
 		(at 238.76 138.43 180)
@@
 		)
 	)
+	(global_label "BK2"
+		(shape input)
+		(at 171.45 101.6 180)
+		(fields_autoplaced yes)
+		(effects
+			(font
+				(size 1.1938 1.1938)
+			)
+			(justify right)
+		)
+		(property "Intersheetrefs" "${INTERSHEET_REFS}"
+			(at 165.7345 101.6 0)
+			(effects
+				(font
+					(size 1.27 1.27)
+				)
+				(justify right)
+				(hide yes)
+			)
+		)
+	)
 	(global_label "PIRQ"
 		(shape output)
@@
 	(global_label "GND"
 		(shape input)
-		(at 153.67 46.99 180)
+		(at 153.67 49.53 180)
 		(fields_autoplaced yes)
 		(effects
@@
 		)
 		(property "Intersheetrefs" "${INTERSHEET_REFS}"
-			(at 95.25 -49.53 0)
+			(at 95.25 -46.99 0)
 			(effects
 				(font
@@
 		)
 	)
+	(global_label "BA16"
+		(shape output)
+		(at 201.93 91.44 0)
+		(fields_autoplaced yes)
+		(effects
+			(font
+				(size 1.1938 1.1938)
+			)
+			(justify left)
+		)
+		(property "Intersheetrefs" "${INTERSHEET_REFS}"
+			(at 208.612 91.44 0)
+			(effects
+				(font
+					(size 1.27 1.27)
+				)
+				(justify left)
+				(hide yes)
+			)
+		)
+	)
 	(global_label "GND"
 		(shape input)
@@
 	(symbol
 		(lib_id "Device:LED")
-		(at 162.56 40.64 90)
+		(at 162.56 43.18 90)
 		(unit 1)
 		(exclude_from_sim no)
@@
 		(dnp no)
 		(property "Reference" "POWER1"
-			(at 165.5572 39.6494 90)
+			(at 165.5572 42.1894 90)
 			(effects
 				(font
@@
 		)
 		(property "Value" "LED (BLUE)"
-			(at 165.5572 41.9608 90)
+			(at 165.5572 44.5008 90)
 			(effects
 				(font
@@
 		)
 		(property "Footprint" "LED_THT:LED_D3.0mm_FlatTop"
-			(at 162.56 40.64 0)
+			(at 162.56 43.18 0)
 			(effects
 				(font
@@
 		)
 		(property "Datasheet" "~"
-			(at 162.56 40.64 0)
+			(at 162.56 43.18 0)
 			(effects
 				(font
@@
 		)
 		(property "Description" "Light emitting diode"
-			(at 162.56 40.64 0)
+			(at 162.56 43.18 0)
 			(effects
 				(font
