File: Schematics/JJ65c02/JJ65c02.kicad_pcb (KiCad board)
At the start: 4 copper layers, 172.7 x 135.9 mm, 53 parts, among them SW2 SW_SPDT, U1 74HC00, U3 TXB0108PWR, U4 TXB0104PW, U6 TLV2217-33KCSE3, X1 1.8Mhz

Commit message: Schematic changes - Banking
Parts:
- CLK1: renamed from SYS CLK
- DECODER1: value 22V10C -> ATF22V10C-7
- R6: value 1.8k -> 2k
- U5: renamed from DATA LATCH
- moved CLK1 7.57 mm to (17.4, 101.6)
- moved SW1 6.84 mm to (21.1, 114.0)
- moved DECODER1 4.98 mm to (22.0, 82.0)
- moved C13 4.98 mm to (16.0, 81.0)
- moved U3 2.56 mm to (91.2, 90.0)
- moved C7 2.06 mm to (24.3, 14.6)
- moved ROM1 1.97 mm to (14.4, 22.7)
- renumbered RESET to SW1
Connections:
- AUDIO1 pad R: Net-(AUDIO1-PadR) -> SND
- AUDIO1 pad T: Net-(AUDIO1-PadR) -> SND
- C11 pad 2: Net-(C11-Pad2) -> SND
- C12 pad 1: Net-(AUDIO1-PadR) -> SND
- C12 pad 2: Net-(C11-Pad2) -> SND
- DECODER1 pad 11: unconnected-(DECODER1-IN11-Pad11) -> BK2
- DECODER1 pad 18: unconnected-(DECODER1-IO17-Pad18) -> BA16
- R4 pad 1: Net-(C11-Pad2) -> SND
- R5 pad 2: Net-(C11-Pad2) -> SND
- R6 pad 2: Net-(AUDIO1-PadR) -> SND
- RAM1 pad 2: BK2 -> BA16
Routing:
- net GND: track 11.2 -> 764.3 mm, vias 4 -> 1
- net SND: track 50.8 -> 123.2 mm
- net Net-(AUDIO1-PadR): track 64.7 -> 0.00 mm
- net BA16: track 0.00 -> 51.5 mm
- net a3: track 125.0 -> 95.2 mm
- net pa3v4: track 93.4 -> 66.0 mm
- net Net-(C11-Pad2): track 25.7 -> 0.00 mm
- net Net-(RN2B-R2.2): track 153.1 -> 128.5 mm, vias 1 -> 0
- net Net-(RAM1-CE2): track 102.6 -> 125.0 mm
- net CLK: track 226.0 -> 207.1 mm
- net d5: track 144.3 -> 161.8 mm, vias 1 -> 2
- net pa3v1: track 94.2 -> 79.3 mm
- net pa3v2: track 85.3 -> 72.0 mm, vias 2 -> 1
- net d0: track 190.2 -> 180.5 mm, vias 2 -> 1
- net Net-(NE1-DIS): track 147.1 -> 156.6 mm, vias 2 -> 1
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- removed copper zone on B.Cu, net GND
